File: wireless.sch (KiCad schematic (older format))
At the start: 18 parts

Commit message: Annotation
Parts:
- gave numbers to parts that had none: 18
Connections:
- wire segments 67 -> 48
Changed lines of the file:
@@
 $Descr A4 11693 8268
 encoding utf-8
-Sheet 4 4
-Title ""
-Date ""
-Rev ""
-Comp ""
-Comment1 ""
+Sheet 3 4
+Title "Speedy the nanocopter autopilot"
+Date "Mon 25 Mai 2015"
+Rev "A"
+Comp "Salah-Eddine Missri"
+Comment1 "License: CC-BY 4.0"
 Comment2 ""
 Comment3 ""
@@
 $EndDescr
 $Comp
-L NRF24R01+ U?
+L NRF24R01+ U7
 U 1 1 55438B0D
 P 5175 3125
-F 0 "U?" H 5175 3125 60  0000 C CNN
+F 0 "U7" H 5175 3125 60  0000 C CNN
 F 1 "NRF24L01+" H 5225 3275 60  0000 C CNN
 F 2 "" H 5175 3125 60  0000 C CNN
@@
 $EndComp
 $Comp
-L VCC #PWR050
+L VCC #PWR056
 U 1 1 55438B1A
 P 3675 2525
-F 0 "#PWR050" H 3675 2375 50  0001 C CNN
+F 0 "#PWR056" H 3675 2375 50  0001 C CNN
 F 1 "VCC" H 3675 2675 50  0000 C CNN
 F 2 "" H 3675 2525 60  0000 C CNN
@@
 $EndComp
 $Comp
-L GND #PWR051
+L GND #PWR057
 U 1 1 55438B20
 P 3675 3475
-F 0 "#PWR051" H 3675 3225 50  0001 C CNN
+F 0 "#PWR057" H 3675 3225 50  0001 C CNN
 F 1 "GND" H 3675 3325 50  0000 C CNN
 F 2 "" H 3675 3475 60  0000 C CNN
@@
 $EndComp
 $Comp
-L R R?
+L R R19
 U 1 1 55438B26
 P 4225 3475
-F 0 "R?" V 4305 3475 50  0000 C CNN
+F 0 "R19" V 4305 3475 50  0000 C CNN
 F 1 "22k" V 4225 3475 50  0000 C CNN
 F 2 "" V 4155 3475 30  0000 C CNN
@@
 $EndComp
 $Comp
-L GND #PWR052
+L GND #PWR058
 U 1 1 55438B2D
 P 4075 4275
-F 0 "#PWR052" H 4075 4025 50  0001 C CNN
+F 0 "#PWR058" H 4075 4025 50  0001 C CNN
 F 1 "GND" H 4075 4125 50  0000 C CNN
 F 2 "" H 4075 4275 60  0000 C CNN
@@
 $EndComp
 $Comp
-L GND #PWR053
+L GND #PWR059
 U 1 1 55438B33
 P 6175 2950
-F 0 "#PWR053" H 6175 2700 50  0001 C CNN
+F 0 "#PWR059" H 6175 2700 50  0001 C CNN
 F 1 "GND" H 6175 2800 50  0000 C CNN
 F 2 "" H 6175 2950 60  0000 C CNN
@@
 $EndComp
 $Comp
-L GND #PWR054
+L GND #PWR060
 U 1 1 55438B39
 P 6525 2950
-F 0 "#PWR054" H 6525 2700 50  0001 C CNN
+F 0 "#PWR060" H 6525 2700 50  0001 C CNN
 F 1 "GND" H 6525 2800 50  0000 C CNN
 F 2 "" H 6525 2950 60  0000 C CNN
@@
 $EndComp
 $Comp
-L L_Small L?
+L L_Small L1
 U 1 1 55438B3F
 P 6025 2525
-F 0 "L?" H 6055 2565 50  0000 L CNN
+F 0 "L1" H 6055 2565 50  0000 L CNN
 F 1 "8.2nH" H 6055 2485 50  0000 L CNN
 F 2 "" H 6025 2525 60  0000 C CNN
@@
 $EndComp
 $Comp
-L L_Small L?
+L L_Small L2
 U 1 1 55438B46
 P 6250 2425
-F 0 "L?" V 6325 2475 50  0000 L CNN
+F 0 "L2" V 6325 2475 50  0000 L CNN
 F 1 "3.9nH" V 6325 2225 50  0000 L CNN
 F 2 "" H 6250 2425 60  0000 C CNN
@@
 $EndComp
 $Comp
-L L_Small L?
+L L_Small L3
 U 1 1 55438B4D
 P 6250 2625
-F 0 "L?" V 6200 2675 50  0000 L CNN
+F 0 "L3" V 6200 2675 50  0000 L CNN
 F 1 "2.7nH" V 6200 2425 50  0000 L CNN
 F 2 "" H 6250 2625 60  0000 C CNN
@@
 $EndComp
 $Comp
-L C_Small C?
+L C_Small C33
 U 1 1 55438B54
 P 6650 2425
-F 0 "C?" V 6725 2475 50  0000 L CNN
+F 0 "C33" V 6725 2475 50  0000 L CNN
 F 1 "1.5pF" V 6725 2175 50  0000 L CNN
 F 2 "" H 6650 2425 60  0000 C CNN
@@
 $EndComp
 $Comp
-L GND #PWR055
+L GND #PWR061
 U 1 1 55438B5B
 P 6900 2675
-F 0 "#PWR055" H 6900 2425 50  0001 C CNN
+F 0 "#PWR061" H 6900 2425 50  0001 C CNN
 F 1 "GND" H 6900 2525 50  0000 C CNN
 F 2 "" H 6900 2675 60  0000 C CNN
@@
 $EndComp
 $Comp
-L C_Small C?
+L C_Small C31
 U 1 1 55438B61
 P 6175 2850
-F 0 "C?" H 6185 2920 50  0000 L CNN
+F 0 "C31" H 6185 2920 50  0000 L CNN
 F 1 "2.2nF" H 6185 2770 50  0000 L CNN
 F 2 "" H 6175 2850 60  0000 C CNN
@@
 $EndComp
 $Comp
-L C_Small C?
+L C_Small C32
 U 1 1 55438B68
 P 6525 2850
-F 0 "C?" H 6535 2920 50  0000 L CNN
+F 0 "C32" H 6535 2920 50  0000 L CNN
 F 1 "4.7pF" H 6535 2770 50  0000 L CNN
 F 2 "" H 6525 2850 60  0000 C CNN
@@
 $EndComp
 $Comp
-L Crystal_Small Y?
+L Crystal_Small Y1
 U 1 1 55438B6F
 P 4075 4000
-F 0 "Y?" H 4075 4100 50  0000 C CNN
+F 0 "Y1" H 4075 4100 50  0000 C CNN
 F 1 "16MHz" H 4075 3900 50  0000 C CNN
 F 2 "" H 4075 4000 60  0000 C CNN
@@
 $EndComp
 $Comp
-L R R?
+L R R18
 U 1 1 55438B76
 P 4075 3725
-F 0 "R?" V 4155 3725 50  0000 C CNN
+F 0 "R18" V 4155 3725 50  0000 C CNN
 F 1 "1M" V 4075 3725 50  0000 C CNN
 F 2 "" V 4005 3725 30  0000 C CNN
@@
 $EndComp
 $Comp
-L C_Small C?
+L C_Small C26
 U 1 1 55438B7D
 P 3775 4150
-F 0 "C?" H 3785 4220 50  0000 L CNN
+F 0 "C26" H 3785 4220 50  0000 L CNN
 F 1 "22pF" H 3785 4070 50  0000 L CNN
 F 2 "" H 3775 4150 60  0000 C CNN
@@
 $EndComp
 $Comp
-L C_Small C?
+L C_Small C30
 U 1 1 55438B84
 P 4375 4150
-F 0 "C?" H 4385 4220 50  0000 L CNN
+F 0 "C30" H 4385 4220 50  0000 L CNN
 F 1 "22pF" H 4385 4070 50  0000 L CNN
 F 2 "" H 4375 4150 60  0000 C CNN
@@
 $EndComp
 $Comp
-L C_Small C?
+L C_Small C27
 U 1 1 55438B8B
 P 3900 3325
-F 0 "C?" V 3950 3200 50  0000 L CNN
+F 0 "C27" V 3950 3200 50  0000 L CNN
 F 1 "33nF" V 3850 3100 50  0000 L CNN
 F 2 "" H 3900 3325 60  0000 C CNN
@@
 $EndComp
 $Comp
-L C_Small C?
+L C_Small C34
 U 1 1 55438B92
 P 6900 2575
-F 0 "C?" H 6910 2645 50  0000 L CNN
+F 0 "C34" H 6910 2645 50  0000 L CNN
 F 1 "1pF" H 6910 2495 50  0000 L CNN
 F 2 "" H 6900 2575 60  0000 C CNN
@@
 $EndComp
 $Comp
-L C_Small C?
+L C_Small C25
 U 1 1 55438B99
 P 3675 2700
-F 0 "C?" H 3685 2770 50  0000 L CNN
+F 0 "C25" H 3685 2770 50  0000 L CNN
 F 1 "0.1uF" H 3685 2620 50  0000 L CNN
 F 2 "" H 3675 2700 60  0000 C CNN
@@
 $EndComp
 $Comp
-L C_Small C?
+L C_Small C29
 U 1 1 55438BA0
 P 4200 2700
-F 0 "C?" H 4210 2770 50  0000 L CNN
+F 0 "C29" H 4210 2770 50  0000 L CNN
 F 1 "1nF" H 4210 2620 50  0000 L CNN
 F 2 "" H 4200 2700 60  0000 C CNN
@@
 $EndComp
 $Comp
-L GND #PWR056
+L GND #PWR062
 U 1 1 55438BA7
 P 3675 2875
-F 0 "#PWR056" H 3675 2625 50  0001 C CNN
+F 0 "#PWR062" H 3675 2625 50  0001 C CNN
 F 1 "GND" H 3675 2725 50  0000 C CNN
 F 2 "" H 3675 2875 60  0000 C CNN
@@
 Connection ~ 4075 4275
 Wire Wire Line
-	3775 4275 4075 4275
-Wire Wire Line
-	4075 4275 4375 4275
+	3775 4275 4375 4275
 Connection ~ 3775 4000
 Connection ~ 4375 4000
@@
 	4425 2625 4375 2625
 Wire Wire Line
-	3675 2525 3950 2525
-Wire Wire Line
-	3950 2525 4200 2525
-Wire Wire Line
-	4200 2525 4375 2525
-Wire Wire Line
-	4375 2525 4425 2525
-Wire Wire Line
-	4375 2525 4375 2625
-Wire Wire Line
-	4375 2625 4375 2725
+	3675 2525 4425 2525
+Wire Wire Line
+	4375 2525 4375 2725
 Wire Wire Line
 	4375 2725 4425 2725
@@
 	4375 3175 4425 3175
 Wire Wire Line
-	4375 2875 4375 2975
-Wire Wire Line
-	4375 2975 4375 3075
-Wire Wire Line
-	4375 3075 4375 3175
-Wire Wire Line
-	3675 2875 3950 2875
-Wire Wire Line
-	3950 2875 4200 2875
-Wire Wire Line
-	4200 2875 4375 2875
-Wire Wire Line
-	4375 2875 4425 2875
-Wire Wire Line
-	3775 3625 3775 3725
-Wire Wire Line
-	3775 3725 3775 4000
-Wire Wire Line
-	3775 4000 3775 4050
+	4375 2875 4375 3175
+Wire Wire Line
+	3675 2875 4425 2875
+Wire Wire Line
+	3775 3625 3775 4050
 Wire Wire Line
 	4425 3625 3775 3625
 Wire Wire Line
-	4375 3725 4375 4000
-Wire Wire Line
-	4375 4000 4375 4050
-Wire Wire Line
-	4225 3725 4375 3725
-Wire Wire Line
-	4375 3725 4425 3725
+	4375 3725 4375 4050
+Wire Wire Line
+	4225 3725 4425 3725
 Wire Wire Line
 	5975 3725 5925 3725
@@
 	5975 3325 5925 3325
 Wire Wire Line
-	6525 2625 6525 2725
-Wire Wire Line
-	6525 2725 6525 2750
-Wire Wire Line
-	5925 2725 6175 2725
-Wire Wire Line
-	6175 2725 6525 2725
+	6525 2625 6525 2750
+Wire Wire Line
+	5925 2725 6525 2725
 Wire Wire Line
 	6175 2725 6175 2750
 Connection ~ 6175 2725
 Wire Wire Line
-	5925 2625 6025 2625
-Wire Wire Line
-	6025 2625 6150 2625
-Wire Wire Line
-	5925 2425 6025 2425
-Wire Wire Line
-	6025 2425 6150 2425
+	5925 2625 6150 2625
+Wire Wire Line
+	5925 2425 6150 2425
 Wire Wire Line
 	6350 2625 6525 2625
@@
 Connection ~ 4200 2875
 $Comp
-L C_Small C?
+L C_Small C28
 U 1 1 55438BFC
 P 3950 2700
-F 0 "C?" H 3960 2770 50  0000 L CNN
+F 0 "C28" H 3960 2770 50  0000 L CNN
 F 1 "10nF" H 3960 2620 50  0000 L CNN
 F 2 "" H 3950 2700 60  0000 C CNN
@@
 Connection ~ 3950 2525
 $Comp
-L ANTENNA A?
+L ANTENNA A1
 U 1 1 55438C07
 P 7475 2625
-F 0 "A?" H 7575 2475 60  0000 C CNN
+F 0 "A1" H 7575 2475 60  0000 C CNN
 F 1 "ANTENNA" H 7475 2925 60  0001 C CNN
 F 2 "" H 7475 2625 60  0000 C CNN
@@
 	6900 2475 6900 2425
 Wire Wire Line
-	6750 2425 6900 2425
-Wire Wire Line
-	6900 2425 7225 2425
+	6750 2425 7225 2425
 Wire Wire Line
 	7475 2925 7225 2925

Commit message: Change MCU to LQFP64 (instead of BGA)
Parts:
- added W10, W11, W12, W13, W8, W9: TEST, symbol TEST
- renumbered C25 to C21, C26 to C22, C27 to C23, C28 to C24, C29 to C25, C30 to C26, C31 to C27, C32 to C28, C33 to C29, C34 to C30, R18 to R17, R19 to R18
Changed lines of the file:
@@
 EESchema Schematic File Version 2
+LIBS:speedy-rescue
 LIBS:speedy-cache
 LIBS:power
@@
 LIBS:memory
 LIBS:xilinx
-LIBS:special
 LIBS:microcontrollers
 LIBS:dsp
@@
 $EndComp
 $Comp
-L VCC #PWR056
+L VCC #PWR043
 U 1 1 55438B1A
 P 3675 2525
-F 0 "#PWR056" H 3675 2375 50  0001 C CNN
+F 0 "#PWR043" H 3675 2375 50  0001 C CNN
 F 1 "VCC" H 3675 2675 50  0000 C CNN
 F 2 "" H 3675 2525 60  0000 C CNN
@@
 $EndComp
 $Comp
-L GND #PWR057
+L GND #PWR044
 U 1 1 55438B20
 P 3675 3475
-F 0 "#PWR057" H 3675 3225 50  0001 C CNN
+F 0 "#PWR044" H 3675 3225 50  0001 C CNN
 F 1 "GND" H 3675 3325 50  0000 C CNN
 F 2 "" H 3675 3475 60  0000 C CNN
@@
 $EndComp
 $Comp
-L R R19
+L R R18
 U 1 1 55438B26
 P 4225 3475
-F 0 "R19" V 4305 3475 50  0000 C CNN
+F 0 "R18" V 4305 3475 50  0000 C CNN
 F 1 "22k" V 4225 3475 50  0000 C CNN
 F 2 "" V 4155 3475 30  0000 C CNN
@@
 $EndComp
 $Comp
-L GND #PWR058
+L GND #PWR045
 U 1 1 55438B2D
 P 4075 4275
-F 0 "#PWR058" H 4075 4025 50  0001 C CNN
+F 0 "#PWR045" H 4075 4025 50  0001 C CNN
 F 1 "GND" H 4075 4125 50  0000 C CNN
 F 2 "" H 4075 4275 60  0000 C CNN
@@
 $EndComp
 $Comp
-L GND #PWR059
+L GND #PWR046
 U 1 1 55438B33
 P 6175 2950
-F 0 "#PWR059" H 6175 2700 50  0001 C CNN
+F 0 "#PWR046" H 6175 2700 50  0001 C CNN
 F 1 "GND" H 6175 2800 50  0000 C CNN
 F 2 "" H 6175 2950 60  0000 C CNN
@@
 $EndComp
 $Comp
-L GND #PWR060
+L GND #PWR047
 U 1 1 55438B39
 P 6525 2950
-F 0 "#PWR060" H 6525 2700 50  0001 C CNN
+F 0 "#PWR047" H 6525 2700 50  0001 C CNN
 F 1 "GND" H 6525 2800 50  0000 C CNN
 F 2 "" H 6525 2950 60  0000 C CNN
@@
 $EndComp
 $Comp
-L C_Small C33
+L C_Small C29
 U 1 1 55438B54
 P 6650 2425
-F 0 "C33" V 6725 2475 50  0000 L CNN
+F 0 "C29" V 6725 2475 50  0000 L CNN
 F 1 "1.5pF" V 6725 2175 50  0000 L CNN
 F 2 "" H 6650 2425 60  0000 C CNN
@@
 $EndComp
 $Comp
-L GND #PWR061
+L GND #PWR048
 U 1 1 55438B5B
 P 6900 2675
-F 0 "#PWR061" H 6900 2425 50  0001 C CNN
+F 0 "#PWR048" H 6900 2425 50  0001 C CNN
 F 1 "GND" H 6900 2525 50  0000 C CNN
 F 2 "" H 6900 2675 60  0000 C CNN
@@
 $EndComp
 $Comp
-L C_Small C31
+L C_Small C27
 U 1 1 55438B61
 P 6175 2850
-F 0 "C31" H 6185 2920 50  0000 L CNN
+F 0 "C27" H 6185 2920 50  0000 L CNN
 F 1 "2.2nF" H 6185 2770 50  0000 L CNN
 F 2 "" H 6175 2850 60  0000 C CNN
@@
 $EndComp
 $Comp
-L C_Small C32
+L C_Small C28
 U 1 1 55438B68
 P 6525 2850
-F 0 "C32" H 6535 2920 50  0000 L CNN
+F 0 "C28" H 6535 2920 50  0000 L CNN
 F 1 "4.7pF" H 6535 2770 50  0000 L CNN
 F 2 "" H 6525 2850 60  0000 C CNN
@@
 $EndComp
 $Comp
-L R R18
+L R R17
 U 1 1 55438B76
 P 4075 3725
-F 0 "R18" V 4155 3725 50  0000 C CNN
+F 0 "R17" V 4155 3725 50  0000 C CNN
 F 1 "1M" V 4075 3725 50  0000 C CNN
 F 2 "" V 4005 3725 30  0000 C CNN
@@
 $EndComp
 $Comp
-L C_Small C26
+L C_Small C22
 U 1 1 55438B7D
 P 3775 4150
-F 0 "C26" H 3785 4220 50  0000 L CNN
+F 0 "C22" H 3785 4220 50  0000 L CNN
 F 1 "22pF" H 3785 4070 50  0000 L CNN
 F 2 "" H 3775 4150 60  0000 C CNN
@@
 $EndComp
 $Comp
-L C_Small C30
+L C_Small C26
 U 1 1 55438B84
 P 4375 4150
-F 0 "C30" H 4385 4220 50  0000 L CNN
+F 0 "C26" H 4385 4220 50  0000 L CNN
 F 1 "22pF" H 4385 4070 50  0000 L CNN
 F 2 "" H 4375 4150 60  0000 C CNN
@@
 $EndComp
 $Comp
-L C_Small C27
+L C_Small C23
 U 1 1 55438B8B
 P 3900 3325
-F 0 "C27" V 3950 3200 50  0000 L CNN
+F 0 "C23" V 3950 3150 50  0000 L CNN
 F 1 "33nF" V 3850 3100 50  0000 L CNN
 F 2 "" H 3900 3325 60  0000 C CNN
@@
 $EndComp
 $Comp
-L C_Small C34
+L C_Small C30
 U 1 1 55438B92
 P 6900 2575
-F 0 "C34" H 6910 2645 50  0000 L CNN
+F 0 "C30" H 6910 2645 50  0000 L CNN
 F 1 "1pF" H 6910 2495 50  0000 L CNN
 F 2 "" H 6900 2575 60  0000 C CNN
@@
 $EndComp
 $Comp
-L C_Small C25
+L C_Small C21
 U 1 1 55438B99
 P 3675 2700
-F 0 "C25" H 3685 2770 50  0000 L CNN
+F 0 "C21" H 3685 2770 50  0000 L CNN
 F 1 "0.1uF" H 3685 2620 50  0000 L CNN
 F 2 "" H 3675 2700 60  0000 C CNN
@@
 $EndComp
 $Comp
-L C_Small C29
+L C_Small C25
 U 1 1 55438BA0
 P 4200 2700
-F 0 "C29" H 4210 2770 50  0000 L CNN
+F 0 "C25" H 4210 2770 50  0000 L CNN
 F 1 "1nF" H 4210 2620 50  0000 L CNN
 F 2 "" H 4200 2700 60  0000 C CNN
@@
 $EndComp
 $Comp
-L GND #PWR062
+L GND #PWR049
 U 1 1 55438BA7
 P 3675 2875
-F 0 "#PWR062" H 3675 2625 50  0001 C CNN
+F 0 "#PWR049" H 3675 2625 50  0001 C CNN
 F 1 "GND" H 3675 2725 50  0000 C CNN
 F 2 "" H 3675 2875 60  0000 C CNN
@@
 	4225 3725 4425 3725
 Wire Wire Line
-	5975 3725 5925 3725
-Wire Wire Line
-	5975 3225 5925 3225
-Wire Wire Line
-	5925 3625 5975 3625
-Wire Wire Line
-	5975 3525 5925 3525
-Wire Wire Line
-	5925 3425 5975 3425
-Wire Wire Line
-	5975 3325 5925 3325
+	6375 3725 6325 3725
+Wire Wire Line
+	6375 3225 6325 3225
+Wire Wire Line
+	6325 3625 6375 3625
+Wire Wire Line
+	6375 3525 6325 3525
+Wire Wire Line
+	6325 3425 6375 3425
+Wire Wire Line
+	6375 3325 6325 3325
 Wire Wire Line
 	6525 2625 6525 2750
@@
 Connection ~ 4200 2875
 $Comp
-L C_Small C28
+L C_Small C24
 U 1 1 55438BFC
 P 3950 2700
-F 0 "C28" H 3960 2770 50  0000 L CNN
+F 0 "C24" H 3960 2770 50  0000 L CNN
 F 1 "10nF" H 3960 2620 50  0000 L CNN
 F 2 "" H 3950 2700 60  0000 C CNN
@@
 Text Notes 7275 2400 0    39   ~ 0
 50ohm 2.4GHz\nRF antenna
-Text HLabel 5975 3225 2    39   Input ~ 0
+Text HLabel 6375 3225 2    39   Input ~ 0
 NRF24L01+_EN
-Text HLabel 5975 3325 2    39   Input ~ 0
+Text HLabel 6375 3325 2    39   Input ~ 0
 NRF24L01+_CS
-Text HLabel 5975 3425 2    39   Input ~ 0
+Text HLabel 6375 3425 2    39   Input ~ 0
 SPI2_SCK
-Text HLabel 5975 3525 2    39   Input ~ 0
+Text HLabel 6375 3525 2    39   Input ~ 0
 SPI2_MOSI
-Text HLabel 5975 3625 2    39   Input ~ 0
+Text HLabel 6375 3625 2    39   Input ~ 0
 SPI2_MISO
-Text HLabel 5975 3725 2    39   Input ~ 0
+Text HLabel 6375 3725 2    39   Input ~ 0
 NRF24L01+_INT
+$Comp
+L TEST W8
+U 1 1 5579456F
+P 6125 3225
+F 0 "W8" H 6275 3250 40  0000 C CNN
+F 1 "TEST" H 6125 3225 20  0000 C CNN
+F 2 "" H 6125 3225 60  0000 C CNN
+F 3 "" H 6125 3225 60  0000 C CNN
+	1    6125 3225
+	1    0    0    -1
+$EndComp
+$Comp
+L TEST W9
+U 1 1 5579499D
+P 6125 3325
+F 0 "W9" H 6275 3350 40  0000 C CNN
+F 1 "TEST" H 6125 3325 20  0000 C CNN
+F 2 "" H 6125 3325 60  0000 C CNN
+F 3 "" H 6125 3325 60  0000 C CNN
+	1    6125 3325
+	1    0    0    -1
+$EndComp
+$Comp
+L TEST W10
+U 1 1 557949DF
+P 6125 3425
+F 0 "W10" H 6275 3450 40  0000 C CNN
+F 1 "TEST" H 6125 3425 20  0000 C CNN
+F 2 "" H 6125 3425 60  0000 C CNN
+F 3 "" H 6125 3425 60  0000 C CNN
+	1    6125 3425
+	1    0    0    -1
+$EndComp
+$Comp
+L TEST W11
+U 1 1 55794A1F
+P 6125 3525
+F 0 "W11" H 6275 3550 40  0000 C CNN
+F 1 "TEST" H 6125 3525 20  0000 C CNN
+F 2 "" H 6125 3525 60  0000 C CNN
+F 3 "" H 6125 3525 60  0000 C CNN
+	1    6125 3525
+	1    0    0    -1
+$EndComp
+$Comp
+L TEST W12
+U 1 1 55794A65
+P 6125 3625
+F 0 "W12" H 6275 3650 40  0000 C CNN
+F 1 "TEST" H 6125 3625 20  0000 C CNN
+F 2 "" H 6125 3625 60  0000 C CNN
+F 3 "" H 6125 3625 60  0000 C CNN
+	1    6125 3625
+	1    0    0    -1
+$EndComp
+$Comp
+L TEST W13
+U 1 1 55794AA9
+P 6125 3725
+F 0 "W13" H 6275 3750 40  0000 C CNN
+F 1 "TEST" H 6125 3725 20  0000 C CNN
+F 2 "" H 6125 3725 60  0000 C CNN
+F 3 "" H 6125 3725 60  0000 C CNN
+	1    6125 3725
+	1    0    0    -1
+$EndComp
 $EndSCHEMATC
