File: wireless.sch (KiCad schematic (older format))
At the start: 24 parts, among them U7 NRF24L01+, Y1 16MHz

Commit message: Netlist
Parts:
- removed Y1: 16MHz, symbol Crystal_Small
- added X2: 16MHz 10ppm, _div:_TSX-3225-SMD-XTAL, symbol XTAL-SMD-4-PADS
- A1: footprint (none) -> _div:_ANT-2.45-CHP
- C21, C22, C23, C24, C25, C26, C27, C28, C29, C30, L1, L2, L3, R17, R18: footprint (none) -> _std:_0402
- U7: footprint (none) -> Housings_DFN_QFN:QFN-20-1EP_4x4mm_Pitch0.5mm
- W10, W11, W12, W13, W8, W9: footprint (none) -> Measurement_Points:Measurement_Point_Square-SMD-Pad_Small
Changed lines of the file:
@@
 F 0 "U7" H 5175 3125 60  0000 C CNN
 F 1 "NRF24L01+" H 5225 3275 60  0000 C CNN
-F 2 "" H 5175 3125 60  0000 C CNN
+F 2 "Housings_DFN_QFN:QFN-20-1EP_4x4mm_Pitch0.5mm" H 5175 3125 60  0001 C CNN
 F 3 "" H 5175 3125 60  0000 C CNN
 	1    5175 3125
@@
 $EndComp
 $Comp
-L VCC #PWR41
+L VCC #PWR041
 U 1 1 55438B1A
 P 3675 2525
-F 0 "#PWR41" H 3675 2375 50  0001 C CNN
+F 0 "#PWR041" H 3675 2375 50  0001 C CNN
 F 1 "VCC" H 3675 2675 50  0000 C CNN
 F 2 "" H 3675 2525 60  0000 C CNN
@@
 $EndComp
 $Comp
-L GND #PWR43
+L GND #PWR042
 U 1 1 55438B20
-P 3675 3475
-F 0 "#PWR43" H 3675 3225 50  0001 C CNN
-F 1 "GND" H 3675 3325 50  0000 C CNN
-F 2 "" H 3675 3475 60  0000 C CNN
-F 3 "" H 3675 3475 60  0000 C CNN
-	1    3675 3475
+P 3275 3475
+F 0 "#PWR042" H 3275 3225 50  0001 C CNN
+F 1 "GND" H 3275 3325 50  0000 C CNN
+F 2 "" H 3275 3475 60  0000 C CNN
+F 3 "" H 3275 3475 60  0000 C CNN
+	1    3275 3475
 	1    0    0    -1
 $EndComp
@@
 F 0 "R18" V 4305 3475 50  0000 C CNN
 F 1 "22k" V 4225 3475 50  0000 C CNN
-F 2 "" V 4155 3475 30  0000 C CNN
+F 2 "_std:_0402" V 4155 3475 30  0001 C CNN
 F 3 "" H 4225 3475 30  0000 C CNN
 	1    4225 3475
@@
 $EndComp
 $Comp
-L GND #PWR44
+L GND #PWR043
 U 1 1 55438B2D
 P 4075 4275
-F 0 "#PWR44" H 4075 4025 50  0001 C CNN
+F 0 "#PWR043" H 4075 4025 50  0001 C CNN
 F 1 "GND" H 4075 4125 50  0000 C CNN
 F 2 "" H 4075 4275 60  0000 C CNN
@@
 $EndComp
 $Comp
-L GND #PWR45
+L GND #PWR044
 U 1 1 55438B33
 P 6175 2950
-F 0 "#PWR45" H 6175 2700 50  0001 C CNN
+F 0 "#PWR044" H 6175 2700 50  0001 C CNN
 F 1 "GND" H 6175 2800 50  0000 C CNN
 F 2 "" H 6175 2950 60  0000 C CNN
@@
 $EndComp
 $Comp
-L GND #PWR46
+L GND #PWR045
 U 1 1 55438B39
 P 6525 2950
-F 0 "#PWR46" H 6525 2700 50  0001 C CNN
+F 0 "#PWR045" H 6525 2700 50  0001 C CNN
 F 1 "GND" H 6525 2800 50  0000 C CNN
 F 2 "" H 6525 2950 60  0000 C CNN
@@
 F 0 "L1" H 6055 2565 50  0000 L CNN
 F 1 "8.2nH" H 6055 2485 50  0000 L CNN
-F 2 "" H 6025 2525 60  0000 C CNN
+F 2 "_std:_0402" H 6025 2525 60  0001 C CNN
 F 3 "" H 6025 2525 60  0000 C CNN
 	1    6025 2525
@@
 F 0 "L2" V 6325 2475 50  0000 L CNN
 F 1 "3.9nH" V 6325 2225 50  0000 L CNN
-F 2 "" H 6250 2425 60  0000 C CNN
+F 2 "_std:_0402" H 6250 2425 60  0001 C CNN
 F 3 "" H 6250 2425 60  0000 C CNN
 	1    6250 2425
@@
 F 0 "L3" V 6200 2675 50  0000 L CNN
 F 1 "2.7nH" V 6200 2425 50  0000 L CNN
-F 2 "" H 6250 2625 60  0000 C CNN
+F 2 "_std:_0402" H 6250 2625 60  0001 C CNN
 F 3 "" H 6250 2625 60  0000 C CNN
 	1    6250 2625
@@
 F 0 "C29" V 6725 2475 50  0000 L CNN
 F 1 "1.5pF" V 6725 2175 50  0000 L CNN
-F 2 "" H 6650 2425 60  0000 C CNN
+F 2 "_std:_0402" H 6650 2425 60  0001 C CNN
 F 3 "" H 6650 2425 60  0000 C CNN
 	1    6650 2425
@@
 $EndComp
 $Comp
-L GND #PWR47
+L GND #PWR046
 U 1 1 55438B5B
 P 6900 2675
-F 0 "#PWR47" H 6900 2425 50  0001 C CNN
+F 0 "#PWR046" H 6900 2425 50  0001 C CNN
 F 1 "GND" H 6900 2525 50  0000 C CNN
 F 2 "" H 6900 2675 60  0000 C CNN
@@
 F 0 "C27" H 6185 2920 50  0000 L CNN
 F 1 "2.2nF" H 6185 2770 50  0000 L CNN
-F 2 "" H 6175 2850 60  0000 C CNN
+F 2 "_std:_0402" H 6175 2850 60  0001 C CNN
 F 3 "" H 6175 2850 60  0000 C CNN
 	1    6175 2850
@@
 F 0 "C28" H 6535 2920 50  0000 L CNN
 F 1 "4.7pF" H 6535 2770 50  0000 L CNN
-F 2 "" H 6525 2850 60  0000 C CNN
+F 2 "_std:_0402" H 6525 2850 60  0001 C CNN
 F 3 "" H 6525 2850 60  0000 C CNN
 	1    6525 2850
-	1    0    0    -1
-$EndComp
-$Comp
-L Crystal_Small Y1
-U 1 1 55438B6F
-P 4075 4000
-F 0 "Y1" H 4075 4100 50  0000 C CNN
-F 1 "16MHz" H 4075 3900 50  0000 C CNN
-F 2 "" H 4075 4000 60  0000 C CNN
-F 3 "" H 4075 4000 60  0000 C CNN
-	1    4075 4000
 	1    0    0    -1
 $EndComp
@@
 F 0 "R17" V 4155 3725 50  0000 C CNN
 F 1 "1M" V 4075 3725 50  0000 C CNN
-F 2 "" V 4005 3725 30  0000 C CNN
+F 2 "_std:_0402" V 4005 3725 30  0001 C CNN
 F 3 "" H 4075 3725 30  0000 C CNN
 	1    4075 3725
@@
 F 0 "C22" H 3785 4220 50  0000 L CNN
 F 1 "22pF" H 3785 4070 50  0000 L CNN
-F 2 "" H 3775 4150 60  0000 C CNN
+F 2 "_std:_0402" H 3775 4150 60  0001 C CNN
 F 3 "" H 3775 4150 60  0000 C CNN
 	1    3775 4150
@@
 F 0 "C26" H 4385 4220 50  0000 L CNN
 F 1 "22pF" H 4385 4070 50  0000 L CNN
-F 2 "" H 4375 4150 60  0000 C CNN
+F 2 "_std:_0402" H 4375 4150 60  0001 C CNN
 F 3 "" H 4375 4150 60  0000 C CNN
 	1    4375 4150
@@
 F 0 "C23" V 3950 3150 50  0000 L CNN
 F 1 "33nF" V 3850 3100 50  0000 L CNN
-F 2 "" H 3900 3325 60  0000 C CNN
+F 2 "_std:_0402" H 3900 3325 60  0001 C CNN
 F 3 "" H 3900 3325 60  0000 C CNN
 	1    3900 3325
@@
 F 0 "C30" H 6910 2645 50  0000 L CNN
 F 1 "1pF" H 6910 2495 50  0000 L CNN
-F 2 "" H 6900 2575 60  0000 C CNN
+F 2 "_std:_0402" H 6900 2575 60  0001 C CNN
 F 3 "" H 6900 2575 60  0000 C CNN
 	1    6900 2575
@@
 F 0 "C21" H 3685 2770 50  0000 L CNN
 F 1 "0.1uF" H 3685 2620 50  0000 L CNN
-F 2 "" H 3675 2700 60  0000 C CNN
+F 2 "_std:_0402" H 3675 2700 60  0001 C CNN
 F 3 "" H 3675 2700 60  0000 C CNN
 	1    3675 2700
@@
 F 0 "C25" H 4210 2770 50  0000 L CNN
 F 1 "1nF" H 4210 2620 50  0000 L CNN
-F 2 "" H 4200 2700 60  0000 C CNN
+F 2 "_std:_0402" H 4200 2700 60  0001 C CNN
 F 3 "" H 4200 2700 60  0000 C CNN
 	1    4200 2700
@@
 $EndComp
 $Comp
-L GND #PWR42
+L GND #PWR047
 U 1 1 55438BA7
 P 3675 2875
-F 0 "#PWR42" H 3675 2625 50  0001 C CNN
+F 0 "#PWR047" H 3675 2625 50  0001 C CNN
 F 1 "GND" H 3675 2725 50  0000 C CNN
 F 2 "" H 3675 2875 60  0000 C CNN
@@
 Connection ~ 3675 3475
 Wire Wire Line
-	3675 3475 4075 3475
+	3275 3475 4075 3475
 Wire Wire Line
 	4425 3475 4375 3475
@@
 Connection ~ 6025 2425
 Connection ~ 6025 2625
-Wire Wire Line
-	3775 4000 3975 4000
-Wire Wire Line
-	4175 4000 4375 4000
 Wire Wire Line
 	3775 4250 3775 4275
@@
 F 0 "C24" H 3960 2770 50  0000 L CNN
 F 1 "10nF" H 3960 2620 50  0000 L CNN
-F 2 "" H 3950 2700 60  0000 C CNN
+F 2 "_std:_0402" H 3950 2700 60  0001 C CNN
 F 3 "" H 3950 2700 60  0000 C CNN
 	1    3950 2700
@@
 F 0 "A1" H 7575 2475 60  0000 C CNN
 F 1 "ANTENNA" H 7475 2925 60  0001 C CNN
-F 2 "" H 7475 2625 60  0000 C CNN
+F 2 "_div:_ANT-2.45-CHP" H 7475 2625 60  0001 C CNN
 F 3 "" H 7475 2625 60  0000 C CNN
 	1    7475 2625
@@
 F 0 "W8" H 6275 3250 40  0000 C CNN
 F 1 "TEST" H 6125 3225 20  0000 C CNN
-F 2 "" H 6125 3225 60  0000 C CNN
+F 2 "Measurement_Points:Measurement_Point_Square-SMD-Pad_Small" H 6125 3225 60  0001 C CNN
 F 3 "" H 6125 3225 60  0000 C CNN
 	1    6125 3225
@@
 F 0 "W9" H 6275 3350 40  0000 C CNN
 F 1 "TEST" H 6125 3325 20  0000 C CNN
-F 2 "" H 6125 3325 60  0000 C CNN
+F 2 "Measurement_Points:Measurement_Point_Square-SMD-Pad_Small" H 6125 3325 60  0001 C CNN
 F 3 "" H 6125 3325 60  0000 C CNN
 	1    6125 3325
@@
 F 0 "W10" H 6275 3450 40  0000 C CNN
 F 1 "TEST" H 6125 3425 20  0000 C CNN
-F 2 "" H 6125 3425 60  0000 C CNN
+F 2 "Measurement_Points:Measurement_Point_Square-SMD-Pad_Small" H 6125 3425 60  0001 C CNN
 F 3 "" H 6125 3425 60  0000 C CNN
 	1    6125 3425
@@
 F 0 "W11" H 6275 3550 40  0000 C CNN
 F 1 "TEST" H 6125 3525 20  0000 C CNN
-F 2 "" H 6125 3525 60  0000 C CNN
+F 2 "Measurement_Points:Measurement_Point_Square-SMD-Pad_Small" H 6125 3525 60  0001 C CNN
 F 3 "" H 6125 3525 60  0000 C CNN
 	1    6125 3525
@@
 F 0 "W12" H 6275 3650 40  0000 C CNN
 F 1 "TEST" H 6125 3625 20  0000 C CNN
-F 2 "" H 6125 3625 60  0000 C CNN
+F 2 "Measurement_Points:Measurement_Point_Square-SMD-Pad_Small" H 6125 3625 60  0001 C CNN
 F 3 "" H 6125 3625 60  0000 C CNN
 	1    6125 3625
@@
 F 0 "W13" H 6275 3750 40  0000 C CNN
 F 1 "TEST" H 6125 3725 20  0000 C CNN
-F 2 "" H 6125 3725 60  0000 C CNN
+F 2 "Measurement_Points:Measurement_Point_Square-SMD-Pad_Small" H 6125 3725 60  0001 C CNN
 F 3 "" H 6125 3725 60  0000 C CNN
 	1    6125 3725
 	1    0    0    -1
 $EndComp
+$Comp
+L XTAL-SMD-4-PADS X2
+U 1 1 558EB9B5
+P 4075 4000
+F 0 "X2" H 4250 3925 60  0000 C CNN
+F 1 "16MHz 10ppm" H 4075 4125 39  0000 C CNN
+F 2 "_div:_TSX-3225-SMD-XTAL" H 4075 4000 60  0001 C CNN
+F 3 "" H 4075 4000 60  0000 C CNN
+	1    4075 4000
+	1    0    0    -1
+$EndComp
+Wire Wire Line
+	4025 4200 4025 4275
+Connection ~ 4025 4275
+Wire Wire Line
+	4125 4200 4125 4275
+Connection ~ 4125 4275
 $EndSCHEMATC

Commit message: Remove CAN interface
(not useful enough, takes too much place)
Parts:
- W10, W11, W12, W13, W8, W9: footprint Measurement_Points:Measurement_Point_Square-SMD-Pad_Small -> _std:Measurement_Point_Round-SMD-Pad_Small
Changed lines of the file:
@@
 F 0 "W8" H 6275 3250 40  0000 C CNN
 F 1 "TEST" H 6125 3225 20  0000 C CNN
-F 2 "Measurement_Points:Measurement_Point_Square-SMD-Pad_Small" H 6125 3225 60  0001 C CNN
+F 2 "_std:Measurement_Point_Round-SMD-Pad_Small" H 6125 3225 60  0001 C CNN
 F 3 "" H 6125 3225 60  0000 C CNN
 	1    6125 3225
@@
 F 0 "W9" H 6275 3350 40  0000 C CNN
 F 1 "TEST" H 6125 3325 20  0000 C CNN
-F 2 "Measurement_Points:Measurement_Point_Square-SMD-Pad_Small" H 6125 3325 60  0001 C CNN
+F 2 "_std:Measurement_Point_Round-SMD-Pad_Small" H 6125 3325 60  0001 C CNN
 F 3 "" H 6125 3325 60  0000 C CNN
 	1    6125 3325
@@
 F 0 "W10" H 6275 3450 40  0000 C CNN
 F 1 "TEST" H 6125 3425 20  0000 C CNN
-F 2 "Measurement_Points:Measurement_Point_Square-SMD-Pad_Small" H 6125 3425 60  0001 C CNN
+F 2 "_std:Measurement_Point_Round-SMD-Pad_Small" H 6125 3425 60  0001 C CNN
 F 3 "" H 6125 3425 60  0000 C CNN
 	1    6125 3425
@@
 F 0 "W11" H 6275 3550 40  0000 C CNN
 F 1 "TEST" H 6125 3525 20  0000 C CNN
-F 2 "Measurement_Points:Measurement_Point_Square-SMD-Pad_Small" H 6125 3525 60  0001 C CNN
+F 2 "_std:Measurement_Point_Round-SMD-Pad_Small" H 6125 3525 60  0001 C CNN
 F 3 "" H 6125 3525 60  0000 C CNN
 	1    6125 3525
@@
 F 0 "W12" H 6275 3650 40  0000 C CNN
 F 1 "TEST" H 6125 3625 20  0000 C CNN
-F 2 "Measurement_Points:Measurement_Point_Square-SMD-Pad_Small" H 6125 3625 60  0001 C CNN
+F 2 "_std:Measurement_Point_Round-SMD-Pad_Small" H 6125 3625 60  0001 C CNN
 F 3 "" H 6125 3625 60  0000 C CNN
 	1    6125 3625
@@
 F 0 "W13" H 6275 3750 40  0000 C CNN
 F 1 "TEST" H 6125 3725 20  0000 C CNN
-F 2 "Measurement_Points:Measurement_Point_Square-SMD-Pad_Small" H 6125 3725 60  0001 C CNN
+F 2 "_std:Measurement_Point_Round-SMD-Pad_Small" H 6125 3725 60  0001 C CNN
 F 3 "" H 6125 3725 60  0000 C CNN
 	1    6125 3725

Commit message: Regenerate netlist & Start placing footprints
Parts:
- removed W10, W11, W12, W13, W8, W9: TEST, _std:Measurement_Point_Round-SMD-Pad_Small, symbol TEST
Connections:
- net NRF24L01+_CS: now also U7.2 (CSN)
- net NRF24L01+_EN: now also U7.1 (CE)
- net NRF24L01+_INT: now also U7.6 (IRQ)
- net SPI2_MISO: now also U7.5 (MISO)
- net SPI2_MOSI: now also U7.4 (MOSI)
- net SPI2_SCK: now also U7.3 (SCK)
Other:
- moved on the sheet: A1
Changed lines of the file:
@@
 EESchema Schematic File Version 2
-LIBS:speedy-rescue
 LIBS:speedy-cache
 LIBS:power
@@
 	4225 3725 4425 3725
 Wire Wire Line
-	6375 3725 6325 3725
-Wire Wire Line
-	6375 3225 6325 3225
-Wire Wire Line
-	6325 3625 6375 3625
-Wire Wire Line
-	6375 3525 6325 3525
-Wire Wire Line
-	6325 3425 6375 3425
-Wire Wire Line
-	6375 3325 6325 3325
+	5975 3725 5925 3725
+Wire Wire Line
+	5975 3225 5925 3225
+Wire Wire Line
+	5925 3625 5975 3625
+Wire Wire Line
+	5975 3525 5925 3525
+Wire Wire Line
+	5925 3425 5975 3425
+Wire Wire Line
+	5975 3325 5925 3325
 Wire Wire Line
 	6525 2625 6525 2750
@@
 L ANTENNA A1
 U 1 1 55438C07
-P 7475 2625
-F 0 "A1" H 7575 2475 60  0000 C CNN
-F 1 "ANTENNA" H 7475 2925 60  0001 C CNN
-F 2 "_div:_ANT-2.45-CHP" H 7475 2625 60  0001 C CNN
-F 3 "" H 7475 2625 60  0000 C CNN
-	1    7475 2625
+P 7475 2125
+F 0 "A1" H 7575 1975 60  0000 C CNN
+F 1 "ANTENNA" H 7475 2425 60  0001 C CNN
+F 2 "_div:_ANT-2.45-CHP" H 7475 2125 60  0001 C CNN
+F 3 "" H 7475 2125 60  0000 C CNN
+	1    7475 2125
 	1    0    0    -1
 $EndComp
@@
 	6900 2475 6900 2425
 Wire Wire Line
-	6750 2425 7225 2425
-Wire Wire Line
-	7475 2925 7225 2925
-Wire Wire Line
-	7225 2925 7225 2425
+	6750 2425 7475 2425
 Connection ~ 6900 2425
-Text Notes 7275 2400 0    39   ~ 0
+Text Notes 7750 2125 0    39   ~ 0
 50ohm 2.4GHz\nRF antenna
-Text HLabel 6375 3225 2    39   Input ~ 0
+Text HLabel 5975 3225 2    39   Input ~ 0
 NRF24L01+_EN
-Text HLabel 6375 3325 2    39   Input ~ 0
+Text HLabel 5975 3325 2    39   Input ~ 0
 NRF24L01+_CS
-Text HLabel 6375 3425 2    39   Input ~ 0
+Text HLabel 5975 3425 2    39   Input ~ 0
 SPI2_SCK
-Text HLabel 6375 3525 2    39   Input ~ 0
+Text HLabel 5975 3525 2    39   Input ~ 0
 SPI2_MOSI
-Text HLabel 6375 3625 2    39   Input ~ 0
+Text HLabel 5975 3625 2    39   Input ~ 0
 SPI2_MISO
-Text HLabel 6375 3725 2    39   Input ~ 0
+Text HLabel 5975 3725 2    39   Input ~ 0
 NRF24L01+_INT
 $Comp
-L TEST W8
-U 1 1 5579456F
-P 6125 3225
-F 0 "W8" H 6275 3250 40  0000 C CNN
-F 1 "TEST" H 6125 3225 20  0000 C CNN
-F 2 "_std:Measurement_Point_Round-SMD-Pad_Small" H 6125 3225 60  0001 C CNN
-F 3 "" H 6125 3225 60  0000 C CNN
-	1    6125 3225
-	1    0    0    -1
-$EndComp
-$Comp
-L TEST W9
-U 1 1 5579499D
-P 6125 3325
-F 0 "W9" H 6275 3350 40  0000 C CNN
-F 1 "TEST" H 6125 3325 20  0000 C CNN
-F 2 "_std:Measurement_Point_Round-SMD-Pad_Small" H 6125 3325 60  0001 C CNN
-F 3 "" H 6125 3325 60  0000 C CNN
-	1    6125 3325
-	1    0    0    -1
-$EndComp
-$Comp
-L TEST W10
-U 1 1 557949DF
-P 6125 3425
-F 0 "W10" H 6275 3450 40  0000 C CNN
-F 1 "TEST" H 6125 3425 20  0000 C CNN
-F 2 "_std:Measurement_Point_Round-SMD-Pad_Small" H 6125 3425 60  0001 C CNN
-F 3 "" H 6125 3425 60  0000 C CNN
-	1    6125 3425
-	1    0    0    -1
-$EndComp
-$Comp
-L TEST W11
-U 1 1 55794A1F
-P 6125 3525
-F 0 "W11" H 6275 3550 40  0000 C CNN
-F 1 "TEST" H 6125 3525 20  0000 C CNN
-F 2 "_std:Measurement_Point_Round-SMD-Pad_Small" H 6125 3525 60  0001 C CNN
-F 3 "" H 6125 3525 60  0000 C CNN
-	1    6125 3525
-	1    0    0    -1
-$EndComp
-$Comp
-L TEST W12
-U 1 1 55794A65
-P 6125 3625
-F 0 "W12" H 6275 3650 40  0000 C CNN
-F 1 "TEST" H 6125 3625 20  0000 C CNN
-F 2 "_std:Measurement_Point_Round-SMD-Pad_Small" H 6125 3625 60  0001 C CNN
-F 3 "" H 6125 3625 60  0000 C CNN
-	1    6125 3625
-	1    0    0    -1
-$EndComp
-$Comp
-L TEST W13
-U 1 1 55794AA9
-P 6125 3725
-F 0 "W13" H 6275 3750 40  0000 C CNN
-F 1 "TEST" H 6125 3725 20  0000 C CNN
-F 2 "_std:Measurement_Point_Round-SMD-Pad_Small" H 6125 3725 60  0001 C CNN
-F 3 "" H 6125 3725 60  0000 C CNN
-	1    6125 3725
-	1    0    0    -1
-$EndComp
-$Comp
 L XTAL-SMD-4-PADS X2
