File: electronics/speedy.sch (KiCad schematic (older format))
At the start: 42 parts, among them SW1 DFU, U1 STM32F415RGT6, U2 NUF2042VX6, X1 16Mhz 10ppm

Commit message: Use wifi for telemetry
Cleanup schematic
Use ESP12E (wifi) for telemetry instead of NRF24
Reannotate & replot pdf
Parts:
- removed D1: POWER, _std:_LED_0603, symbol LED-RESCUE-speedy
- removed D2: ERROR, _std:_LED_0603, symbol LED-RESCUE-speedy
- removed D3: STATUS, _std:_LED_0603, symbol LED-RESCUE-speedy
- removed D4: HEARTBEAT, _std:_LED_0603, symbol LED-RESCUE-speedy
- removed R13, R14, R15, R16: 1k, _std:_0402, symbol R
- removed R6, R8: 10k, _std:_0402, symbol R
- added C12: 0.1uF, _std:_0402, symbol C_Small
- added C13: 100uF, _std:_0603, symbol C_Small
- added D2: POWER, _std:_LED_0603, symbol Led_Small
- added D3: ERROR, _std:_LED_0603, symbol Led_Small
- added D4: STATUS, _std:_LED_0603, symbol Led_Small
- added D5: DEBUG, _std:_LED_0603, symbol Led_Small
- added R12, R9: 10k, _std:_0402, symbol R
- added R4, R5, R6: 10k, _std:_0402, symbol R_Small
- added RP1: 1k, Resistors_SMD:R_Array_Concave_4x0402, symbol R_PACK4
- added U3: ESP-12E, _esp:ESP-12-E, symbol ESP-12E
- added W1: IMU_CS, _div:TestPad, symbol TEST
- added W2: IMU_SCK, _div:TestPad, symbol TEST
- added W3: IMU_MISO, _div:TestPad, symbol TEST
- added W4: IMU_MOSI, _div:TestPad, symbol TEST
- CONN3: renamed from CONN2; footprint _div:_Molex-microSD-WM6701 -> _div:_Molex-microSD-502570-0893
- F1: value 500mA -> 0ZCJ0050AF2E
- U2: renamed from U1; value STM32F415RGT6 -> STM32F405RGT6
- renumbered C3 to C1, C5 to C10, C9 to C11, C10 to C14, C11 to C15, C1 to C2, C2 to C3, C6 to C5, C12 to C6, C13 to C7, C7 to C8, C8 to C9, CONN3 to CONN1, CONN1 to CONN2, D5 to D1, R4 to R1, R12 to R13, R3 to R14, R5 to R15, R7 to R2, R9 to R3, R2 to R7, R1 to R8, U2 to U1
Connections:
- net ERROR_LED: now also RP1.2 (P2)
- net GND: now also C12.2, C13.2, D2.1 (K), D3.1 (K), D4.1 (K), D5.1 (K), R6.1, U3.15 (GND)
- net SDIO_D0: now also R9.2
- net SDIO_D1: now also R10.2
- net SDIO_D2: now also R11.2; no longer R10.2
- net SDIO_D3: now also R12.2; no longer R11.2
- net STATUS_LED: now also RP1.3 (P3)
- net VCC: now also C13.1, R12.1, R4.1, R5.1, R9.1, RP1.1 (P1), U3.8 (VDD)
- net HEARTBEAT_LED renamed DEBUG_LED
- net DEBUG_LED: now also RP1.4 (P4)
- net MCU_OSC_OUT renamed WIFI_RST_N
- net WIFI_RST_N: now also C12.1, U3.1 (~RST)
- net MPU9250_CS: no longer names the net of U2.20 (PA4)
- net MPU9250_CS: now also W1.1
- net MPU9250_INT renamed IMU_INT
- net NRF24L01+_CS renamed WIFI_CS
- net WIFI_CS: now also U3.12 (CS0)
- net NRF24L01+_EN renamed WIFI_EN
- net WIFI_EN: now also U3.3 (EN)
- net NRF24L01+_INT renamed WIFI_INT
- net WIFI_INT: now also U3.13 (INT)
- net SENSOR_PWR_ON renamed SENSOR_PWR_EN
- net SPI1_MISO: no longer names the net of U2.22 (PA6)
- net SPI1_MISO: now also W3.1
- net SPI1_MOSI: no longer names the net of U2.23 (PA7)
- net SPI1_MOSI: now also W4.1
- net SPI1_SCK: no longer names the net of U2.21 (PA5)
- net SPI1_SCK: now also W2.1
- net SPI2_MISO renamed WIFI_MISO
- net WIFI_MISO: now also U3.10 (MISO)
- net SPI2_MOSI renamed WIFI_MOSI
- net WIFI_MOSI: now also U3.9 (MOSI)
- net SPI2_SCK renamed WIFI_SCK
- net WIFI_SCK: now also U3.14 (SCLK)
- net V_USB renamed +5V_protected
- new net: R6.2, U3.16 (GPIO15)
- new net: R5.2, U3.17 (GPIO2)
- new net: R4.2, U3.18 (GPIO0/CS2)
- new net: D5.2 (A), RP1.5 (R4)
- new net: D4.2 (A), RP1.6 (R3)
- new net: D3.2 (A), RP1.7 (R2)
- new net: D2.2 (A), RP1.8 (R1)
- new net IMU_CS: W1.2
- new net IMU_MISO: W3.2
- new net IMU_MOSI: W4.2
- new net IMU_SCK: W2.2
- no-connect marks 2 -> 12
Other:
- note added: "Debug interface"
- note added: "SD card"
- note added: "SPI 1"
- note added: "SPI 2"
- note added: "USB"
- note added: "WIFI"
- note removed: "SD Card interface"
- note removed: "SPI 1 used for \nMPU9250"
- note removed: "SPI 2 used for \nNRF24L01+"
- note removed: "SWD interface"
- note removed: "USB Termination"
- moved on the sheet: C6, C7, CONN1, CONN2, CONN3, D1, F1, R2, R3, U1

Commit message: Update with small corrections
Decrease LED resistor values
Fix NUF2042 name
Fix MPU9250 wiring (contradictory datasheet)
Parts:
- removed U1: NUF2042VX6, _std:SOT-563_6-lead, symbol NUF2042VX6
- added U1: NUF2042XV6, _std:SOT-563_6-lead, symbol NUF2042XV6
- RP1: value 1k -> 330
Connections:
- net +5V_protected: now also U1.5 (VBUS)
- net GND: now also U1.2 (GND)
- net USB_DM: now also U1.3 (DM_I)
- net USB_DP: now also U1.1 (DP_I)
- net at CONN1.2 (D-): now also U1.4 (DM_O)
- net at CONN1.3 (D+): now also U1.6 (DP_O)
Changed lines of the file:
@@
 WIFI_INT
-$Comp
-L NUF2042VX6 U1
-U 1 1 554415CC
-P 6925 1275
-F 0 "U1" H 7175 825 60  0000 C CNN
-F 1 "NUF2042VX6" H 6925 1625 60  0000 C CNN
-F 2 "_std:SOT-563_6-lead" H 6925 925 60  0001 C CNN
-F 3 "" H 6925 925 60  0000 C CNN
-	1    6925 1275
-	1    0    0    -1
-$EndComp
 $Comp
 L GND #PWR012
@@
 P 7100 6250
 F 0 "RP1" H 7100 6775 50  0000 C CNN
-F 1 "1k" H 7100 6700 50  0000 C CNN
+F 1 "330" H 7100 6700 50  0000 C CNN
 F 2 "Resistors_SMD:R_Array_Concave_4x0402" H 7100 6250 50  0001 C CNN
 F 3 "" H 7100 6250 50  0000 C CNN
@@
 	4575 5325 4575 5350
 Connection ~ 4725 5325
+$Comp
+L NUF2042XV6 U1
+U 1 1 576F4472
+P 6925 1275
+F 0 "U1" H 6925 1762 60  0000 C CNN
+F 1 "NUF2042XV6" H 6925 1656 60  0000 C CNN
+F 2 "_std:SOT-563_6-lead" H 6925 925 60  0001 C CNN
+F 3 "" H 6925 925 60  0000 C CNN
+	1    6925 1275
+	1    0    0    -1
+$EndComp
 $EndSCHEMATC

Commit message: Finish routing
Parts:
- C13, C6: footprint _std:_0603 -> _std:C_0603
- D2, D3, D4, D5: footprint _std:_LED_0603 -> _std:D_0603
Connections:
- net DEBUG_LED: now also U2.16 (PA2); no longer U2.11 (PC3)
- net ERROR_LED: now also U2.14 (PA0_WKUP); no longer U2.9 (PC1)
- net IR_EN_BOTTOM: now also U2.41 (PA8); no longer U2.62 (PB9)
- net MOTOR_1_EN: now also U2.10 (PC2); no longer U2.26 (PB0)
- net MOTOR_2_EN: now also U2.11 (PC3); no longer U2.27 (PB1)
- net MOTOR_4_EN: now also U2.9 (PC1); no longer U2.57 (PB5)
- net POWER_KILL: now also U2.26 (PB0); no longer U2.15 (PA1)
- net PUSHBUTTON_INT: now also U2.27 (PB1); no longer U2.16 (PA2)
- net STATUS_LED: now also U2.15 (PA1); no longer U2.10 (PC2)
- net TOF_GPIO1: now also U2.62 (PB9); no longer U2.50 (PA15)
- net TOF_XSHUT: now also U2.57 (PB5); no longer U2.14 (PA0_WKUP)
- net WIFI_RST_N: now also U2.50 (PA15); no longer U2.41 (PA8)
Changed lines of the file:
@@
 Text Label 11000 6025 2    39   ~ 0
 MOTOR_4_IN
-Text Label 4400 3250 2    39   ~ 0
+Text Label 4400 5150 2    39   ~ 0
 MOTOR_1_EN
-Text Label 4400 3350 2    39   ~ 0
+Text Label 4400 5250 2    39   ~ 0
 MOTOR_2_EN
 Text Label 4400 6450 2    39   ~ 0
 MOTOR_3_EN
-Text Label 4400 3750 2    39   ~ 0
+Text Label 4400 5050 2    39   ~ 0
 MOTOR_4_EN
 Text Label 4400 2450 2    39   ~ 0
@@
 F 0 "C6" H 6630 2625 50  0000 L CNN
 F 1 "10uF" H 6630 2500 50  0000 L CNN
-F 2 "_std:_0603" H 6605 2575 60  0001 C CNN
+F 2 "_std:C_0603" H 6605 2575 60  0001 C CNN
 F 3 "" H 6605 2575 60  0000 C CNN
 	1    6605 2575
@@
 Text Label 11000 4500 2    39   ~ 0
 POWER_KILL
-Text Label 4400 1750 2    39   ~ 0
+Text Label 4400 3350 2    39   ~ 0
 PUSHBUTTON_INT
-Text Label 4400 1650 2    39   ~ 0
+Text Label 4400 3250 2    39   ~ 0
 POWER_KILL
 Text Label 11000 4700 2    39   ~ 0
@@
 Text Label 4400 4050 2    39   ~ 0
 IR_EN_TOP
-Text Label 4400 4150 2    39   ~ 0
+Text Label 4400 2350 2    39   ~ 0
 IR_EN_BOTTOM
 $Comp
@@
 Text Label 6525 6200 0    39   ~ 0
 DEBUG_LED
-Text Label 4400 5050 2    39   ~ 0
+Text Label 4400 1550 2    39   ~ 0
 ERROR_LED
-Text Label 4400 5150 2    39   ~ 0
+Text Label 4400 1650 2    39   ~ 0
 STATUS_LED
-Text Label 4400 5250 2    39   ~ 0
+Text Label 4400 1750 2    39   ~ 0
 DEBUG_LED
 Text Notes 650  975  0    60   ~ 0
@@
 Text Label 10700 3300 2    39   ~ 0
 TOF_XSHUT
-Text Label 4400 1550 2    39   ~ 0
+Text Label 4400 3750 2    39   ~ 0
 TOF_XSHUT
-Text Label 4400 3050 2    39   ~ 0
+Text Label 4400 4150 2    39   ~ 0
 TOF_GPIO1
 Text Label 4400 4450 2    39   ~ 0
@@
 Text Label 4400 3550 2    39   ~ 0
 WIFI_INT
-Text Label 4400 2350 2    39   ~ 0
+Text Label 4400 3050 2    39   ~ 0
 WIFI_RST_N
 Text Notes 4775 2125 0    39   ~ 0
@@
 F 0 "D2" H 7575 5875 50  0000 C CNN
 F 1 "POWER" H 7850 5875 50  0000 C CNN
-F 2 "_std:_LED_0603" V 7675 5900 50  0001 C CNN
+F 2 "_std:D_0603" V 7675 5900 50  0001 C CNN
 F 3 "" V 7675 5900 50  0000 C CNN
 	1    7675 5900
@@
 F 0 "D3" H 7575 5975 50  0000 C CNN
 F 1 "ERROR" H 7850 5975 50  0000 C CNN
-F 2 "_std:_LED_0603" V 7675 6000 50  0001 C CNN
+F 2 "_std:D_0603" V 7675 6000 50  0001 C CNN
 F 3 "" V 7675 6000 50  0000 C CNN
 	1    7675 6000
@@
 F 0 "D4" H 7575 6075 50  0000 C CNN
 F 1 "STATUS" H 7850 6075 50  0000 C CNN
-F 2 "_std:_LED_0603" V 7675 6100 50  0001 C CNN
+F 2 "_std:D_0603" V 7675 6100 50  0001 C CNN
 F 3 "" V 7675 6100 50  0000 C CNN
 	1    7675 6100
@@
 F 0 "D5" H 7575 6175 50  0000 C CNN
 F 1 "DEBUG" H 7850 6175 50  0000 C CNN
-F 2 "_std:_LED_0603" V 7675 6200 50  0001 C CNN
+F 2 "_std:D_0603" V 7675 6200 50  0001 C CNN
 F 3 "" V 7675 6200 50  0000 C CNN
 	1    7675 6200
@@
 	10275 1475 9600 1475
 Wire Wire Line
-	4400 3750 3825 3750
+	4400 5050 3825 5050
 Wire Wire Line
 	9600 1575 10275 1575
@@
 	4400 2850 3825 2850
 Wire Wire Line
-	3825 5050 4400 5050
+	3825 1550 4400 1550
 Wire Wire Line
 	4400 4950 3825 4950
@@
 	4400 5650 3825 5650
 Wire Wire Line
+	4400 5250 3825 5250
+Wire Wire Line
+	4400 5150 3825 5150
+Wire Wire Line
+	3825 3050 4400 3050
+Wire Wire Line
+	4400 2450 3825 2450
+Wire Wire Line
+	4400 2550 3825 2550
+Wire Wire Line
 	4400 3350 3825 3350
-Wire Wire Line
-	4400 3250 3825 3250
-Wire Wire Line
-	3825 2350 4400 2350
-Wire Wire Line
-	4400 2450 3825 2450
-Wire Wire Line
-	4400 2550 3825 2550
-Wire Wire Line
-	4400 1750 3825 1750
 Wire Wire Line
 	4400 6350 3825 6350
@@
 	5675 500  5675 7825
 Wire Wire Line
-	4400 5250 3825 5250
-Wire Wire Line
-	4400 5150 3825 5150
+	4400 1750 3825 1750
+Wire Wire Line
+	4400 1650 3825 1650
 Wire Wire Line
 	4400 6250 3825 6250
@@
 	4400 5350 3825 5350
 Wire Wire Line
-	4400 4150 3825 4150
+	4400 2350 3825 2350
 Wire Wire Line
 	4400 4050 3825 4050
@@
 Connection ~ 1850 5400
 Wire Wire Line
-	3825 1650 4400 1650
+	3825 3250 4400 3250
 Wire Wire Line
 	5775 3850 6625 3850
@@
 	10350 3200 10700 3200
 Wire Wire Line
-	3825 1550 4400 1550
-Wire Wire Line
-	4400 3050 3825 3050
+	3825 3750 4400 3750
+Wire Wire Line
+	4400 4150 3825 4150
 Wire Notes Line
 	4425 4775 4450 4775
@@
 F 0 "C13" H 6475 4525 50  0000 L CNN
 F 1 "100uF" H 6475 4375 50  0000 L CNN
-F 2 "_std:_0603" H 6450 4450 60  0001 C CNN
+F 2 "_std:C_0603" H 6450 4450 60  0001 C CNN
 F 3 "" H 6450 4450 60  0000 C CNN
 	1    6450 4450
